File: Proyecto.sch (KiCad schematic (older format))
At the start: 40 parts, among them J10 PORTC, J11 PORTE, J12 Pickit 3, J2 Alimentacion, J3 LCD, J4 Teclado, J5 hc-06, J6 PORTA, J7 Vusb, J8 PORTB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

Commit message: Correccion 1.0
Parts:
- removed SW1: Power/Acticidad/Cuidado, Button_Switch_THT:SW_DIP_SPSTx04_Piano_10.8x11.72mm_W7.62mm_P2.54mm, symbol Switch:SW_DIP_x04
- added C5, C6, C7, C8: CAP, Capacitor_THT:CP_Radial_D5.0mm_P2.00mm, symbol pspice:CAP
- added R13, R15: R, Resistor_THT:R_Axial_DIN0207_L6.3mm_D2.5mm_P7.62mm_Horizontal, symbol Device:R
- added SW1: SW_Push_Dual_x2, Button_Switch_THT:SW_PUSH_6mm, symbol Switch:SW_Push_Dual_x2
Connections:
- net VCC is gone; now on net 12v: J2.1
- net GND: now also C5.2, C6.2, C7.2, C8.2; no longer C1.2
- net MCRLF: now also R15.1
- net Vusb: now also C5.1
- net PIN32: now reaches U3.32 (VDD)
- net PIN32: now also C7.1
- net V renamed PIN11
- net PIN11: now also C6.1, R13.2
- net V4 renamed 12v
- net 12v: no longer C1.1
- new net: R13.1, R15.2, SW1.1 (C)
- new net: C8.1, SW1.2 (D)
- no-connect marks 6 -> 7
Other:
- moved on the sheet: C2, C3, C4, D5, U2, U4
